File: hardware/pcb/kicad/racing_sensor_board.kicad_sch (KiCad schematic)
At the start: 120 parts, among them J0 TC0_Conn, J1 TC1_Conn, J10 NTC2_IN, J11 NTC3_IN, J12 LOAD0, J13 LOAD1, J14 LOAD2, J15 LOAD3, J16 ANA0_IN, J17 ANA1_IN, J18 ANA2_IN, J19 ANA3_IN, J2 TC2_Conn, J20 ANA4_IN, J21 ANA5_IN, J22 ANA6_IN, J23 ANA7_IN, J24 DIG0_IN, J25 DIG1_IN, J26 DIG2_IN, J27 DIG3_IN, J28 DIG4_IN, J29 DIG5_IN, J3 TC3_Conn, J30 12V_IN, J4 TC4_Conn, J5 TC5_Conn, J6 TC6_Conn, J7 TC7_Conn, J8 NTC0_IN, J9 NTC1_IN, Q1 AO3400A, Q2 AO3400A, Q3 AO3400A, Q4 AO3400A, U1 MP2307DN_5V, U10 MAX31855KASA, U2 Teensy41, U3 MAX31855KASA, U4 MAX31855KASA, U5 MAX31855KASA, U6 MAX31855KASA, U7 MAX31855KASA, U8 MAX31855KASA, U9 MAX31855KASA

Commit message: Replace net labels with numbers (dot-to-dot system) in KiCad schematic
All 58 signal nets now use numbers (1-58) instead of descriptive names.
Same number on both ends = same wire, like a dot-to-dot puzzle:
  1=SPI_MOSI, 2=SPI_MISO, 3=SPI_SCK ... 58=TC7_MINUS

Legend table added directly to schematic (bottom-left).
Added KABELKART.md with full printable wiring reference showing
every number, net name, and which component pins connect.

Power nets (GND/+5V/+3V3/+12V) keep descriptive names.

https://claude.ai/code/session_01NVvsy3kMr9piDWfs5WdvpG
Connections:
- net ANA0 renamed 30
- net ANA1 renamed 31
- net ANA2 renamed 32
- net ANA3 renamed 33
- net ANA4 renamed 34
- net ANA5 renamed 35
- net ANA6 renamed 36
- net ANA7 renamed 37
- net CS_ACC renamed 8
- net CS_ETH renamed 7
- net CS_TC0 renamed 9
- net CS_TC1 renamed 10
- net CS_TC2 renamed 11
- net CS_TC3 renamed 12
- net CS_TC4 renamed 13
- net CS_TC5 renamed 14
- net CS_TC6 renamed 15
- net CS_TC7 renamed 16
- net DIG0 renamed 20
- net DIG1 renamed 21
- net DIG2 renamed 22
- net DIG3 renamed 23
- net DIG4 renamed 24
- net DIG5 renamed 25
- net INT1_ACC renamed 19
- net INT_ETH renamed 17
- net LED_PIN renamed 42
- net MOS0 renamed 26
- net MOS1 renamed 27
- net MOS2 renamed 28
- net MOS3 renamed 29
- net NTC0 renamed 38
- net NTC1 renamed 39
- net NTC2 renamed 40
- net NTC3 renamed 41
- net RST_ETH renamed 18
- net SP1_MISO renamed 5
- net SP1_MOSI renamed 4
- net SP1_SCK renamed 6
- net SPI_MISO renamed 2
- net SPI_MOSI renamed 1
- net SPI_SCK renamed 3
- net TC0_MINUS renamed 51
- net TC0_PLUS renamed 43
- net TC1_MINUS renamed 52
- net TC1_PLUS renamed 44
- net TC2_MINUS renamed 53
- net TC2_PLUS renamed 45
- net TC3_MINUS renamed 54
- net TC3_PLUS renamed 46
- net TC4_MINUS renamed 55
- net TC4_PLUS renamed 47
- net TC5_MINUS renamed 56
- net TC5_PLUS renamed 48
- net TC6_MINUS renamed 57
- net TC6_PLUS renamed 49
- net TC7_MINUS renamed 58
- net TC7_PLUS renamed 50
Other:
- note added: "10=CS_TC1 | 30=ANA0 | 50=TC7_PLUS"
- note added: "11=CS_TC2 | 31=ANA1 | 51=TC0_MINUS"
- note added: "12=CS_TC3 | 32=ANA2 | 52=TC1_MINUS"
- note added: "13=CS_TC4 | 33=ANA3 | 53=TC2_MINUS"
- note added: "14=CS_TC5 | 34=ANA4 | 54=TC3_MINUS"
- note added: "15=CS_TC6 | 35=ANA5 | 55=TC4_MINUS"
- note added: "16=CS_TC7 | 36=ANA6 | 56=TC5_MINUS"
- note added: "17=INT_ETH | 37=ANA7 | 57=TC6_MINUS"
- note added: "18=RST_ETH | 38=NTC0 | 58=TC7_MINUS"
- note added: "19=INT1_ACC | 39=NTC1"
- note added: "1=SPI_MOSI | 21=DIG1 | 41=NTC3"
- note added: "20=DIG0 | 40=NTC2"
- note added: "2=SPI_MISO | 22=DIG2 | 42=LED_PIN"
- note added: "3=SPI_SCK | 23=DIG3 | 43=TC0_PLUS"
- note added: "4=SP1_MOSI | 24=DIG4 | 44=TC1_PLUS"
- note added: "5=SP1_MISO | 25=DIG5 | 45=TC2_PLUS"
- note added: "6=SP1_SCK | 26=MOS0 | 46=TC3_PLUS"
- note added: "7=CS_ETH | 27=MOS1 | 47=TC4_PLUS"
- note added: "8=CS_ACC | 28=MOS2 | 48=TC5_PLUS"
- note added: "9=CS_TC0 | 29=MOS3 | 49=TC6_PLUS"
- note added: "GND=Jord +5V=+5V +3V3=3.3V +12V=+12V (beholdt som navn, ikke tall)"
- note added: "KABELKART / NET LEGEND"
- note added: "Nr = Nett | Nr = Nett | Nr = Nett"
