File: hardware/pcb/kicad/racing_sensor_board_v0.5.kicad_sch (KiCad schematic)
At the start: 51 parts, among them Q1 AO3400A, Q2 AO3400A, Q3 AO3400A, Q4 AO3400A, U1 Teensy_4.1, U10 MAX31855KASA+, U11 LIS3DH, U12 LMR33630ADDAR, U13 74AHCT125D-Q100, U2 WIZ850io, U3 MAX31855KASA+, U4 MAX31855KASA+, U5 MAX31855KASA+, U6 MAX31855KASA+, U7 MAX31855KASA+, U8 MAX31855KASA+, U9 MAX31855KASA+

Commit message: Add all discrete components to v0.5 schematic (120 total)
Extended gen_kicad_v05.py to emit all ~70 discrete components that were
previously only mentioned in text annotations:
- Buck converter passives: L1, C1-C5, R23-R24 (FB divider)
- RPM two-stage protection: R1 (1.5k), D6 (5.1V Zener), R2 (270), R3 (pull-up)
- DIG1-3 protection: R4-R9 (series + pull-up), D7-D9 (3.3V Zener), C18-C20
- Analog dividers: R10-R13 (10k/15k), C21-C22 (filter)
- NTC pull-ups: R14-R17 (10k), C23-C26 (filter)
- MOSFET gate resistors: R18-R21 (100), PMOS pull-down R22 (10k)
- Bypass caps: C6-C13 (MAX31855), C14-C15 (LIS3DH), C16-C17 (opto/buffer)
- NeoPixel series R25 (300), Status LED R26 (1k) + LED1, Reset SW1
- Test pads TP1-TP10

Also: standard ref designators (R1/C1/J1), p2 dedicated to STATUS_LED,
expansion header updated to 5-pin + GND, deleted WT32-ETH01 footprint,
added REVIEW_ANSWERS.md with answers to all design review blockers.

Co-Authored-By: Claude Sonnet 4.6 <noreply@anthropic.com>
Claude-Session: https://claude.ai/code/session_01NVvsy3kMr9piDWfs5WdvpG
Parts:
- removed D_MOS1, D_MOS2, D_MOS3, D_MOS4: SS14, Diode_SMD:D_SMA, symbol Custom:SS14
- removed D_TVS: SMBJ18A, Diode_SMD:D_SMB, symbol Custom:TVS
- removed J_ANA1: ANA1, TerminalBlock_Phoenix:TerminalBlock_Phoenix_PT-1,5-2-3.5_1x02_P3.50mm_Horizontal, symbol Custom:Conn2pin
- removed J_ANA2: ANA2, TerminalBlock_Phoenix:TerminalBlock_Phoenix_PT-1,5-2-3.5_1x02_P3.50mm_Horizontal, symbol Custom:Conn2pin
- removed J_DIG1: DIG1, TerminalBlock_Phoenix:TerminalBlock_Phoenix_PT-1,5-2-3.5_1x02_P3.50mm_Horizontal, symbol Custom:Conn2pin
- removed J_DIG2: DIG2, TerminalBlock_Phoenix:TerminalBlock_Phoenix_PT-1,5-2-3.5_1x02_P3.50mm_Horizontal, symbol Custom:Conn2pin
- removed J_DIG3: DIG3, TerminalBlock_Phoenix:TerminalBlock_Phoenix_PT-1,5-2-3.5_1x02_P3.50mm_Horizontal, symbol Custom:Conn2pin
- removed J_EXP: EXPANSION, Connector_PinHeader_2.54mm:PinHeader_1x06_P2.54mm_Vertical, symbol Custom:Conn6pin
- removed J_GPS: GPS_MODULE, TerminalBlock_Phoenix:TerminalBlock_Phoenix_PT-1,5-4-3.5_1x04_P3.50mm_Horizontal, symbol Custom:Conn4pin
- removed J_NEO: NEOPIXEL_WS2812B, TerminalBlock_Phoenix:TerminalBlock_Phoenix_PT-1,5-3-3.5_1x03_P3.50mm_Horizontal, symbol Custom:Conn3pin
- removed J_NTC1: NTC1, TerminalBlock_Phoenix:TerminalBlock_Phoenix_PT-1,5-2-3.5_1x02_P3.50mm_Horizontal, symbol Custom:Conn2pin
- removed J_NTC2: NTC2, TerminalBlock_Phoenix:TerminalBlock_Phoenix_PT-1,5-2-3.5_1x02_P3.50mm_Horizontal, symbol Custom:Conn2pin
- removed J_NTC3: NTC3, TerminalBlock_Phoenix:TerminalBlock_Phoenix_PT-1,5-2-3.5_1x02_P3.50mm_Horizontal, symbol Custom:Conn2pin
- removed J_NTC4: NTC4, TerminalBlock_Phoenix:TerminalBlock_Phoenix_PT-1,5-2-3.5_1x02_P3.50mm_Horizontal, symbol Custom:Conn2pin
- removed J_OUT1: OUT1_FAN, TerminalBlock_Phoenix:TerminalBlock_Phoenix_PT-1,5-2-3.5_1x02_P3.50mm_Horizontal, symbol Custom:Conn2pin
- removed J_OUT2: OUT2_PUMP, TerminalBlock_Phoenix:TerminalBlock_Phoenix_PT-1,5-2-3.5_1x02_P3.50mm_Horizontal, symbol Custom:Conn2pin
- removed J_OUT3: OUT3_SHIFT_LIGHT, TerminalBlock_Phoenix:TerminalBlock_Phoenix_PT-1,5-2-3.5_1x02_P3.50mm_Horizontal, symbol Custom:Conn2pin
- removed J_OUT4: OUT4_SPARE, TerminalBlock_Phoenix:TerminalBlock_Phoenix_PT-1,5-2-3.5_1x02_P3.50mm_Horizontal, symbol Custom:Conn2pin
- removed J_PWR: PWR_IN_12V, TerminalBlock_Phoenix:TerminalBlock_Phoenix_MKDS-1,5-2_1x02_P5.08mm_Horizontal, symbol Custom:PwrConn
- removed J_RPM: RPM_IN, TerminalBlock_Phoenix:TerminalBlock_Phoenix_PT-1,5-2-3.5_1x02_P3.50mm_Horizontal, symbol Custom:Conn2pin
- removed J_TC1: TC1, TerminalBlock_Phoenix:TerminalBlock_Phoenix_PT-1,5-2-3.5_1x02_P3.50mm_Horizontal, symbol Custom:Conn2pin
- removed J_TC2: TC2, TerminalBlock_Phoenix:TerminalBlock_Phoenix_PT-1,5-2-3.5_1x02_P3.50mm_Horizontal, symbol Custom:Conn2pin
- removed J_TC3: TC3, TerminalBlock_Phoenix:TerminalBlock_Phoenix_PT-1,5-2-3.5_1x02_P3.50mm_Horizontal, symbol Custom:Conn2pin
- removed J_TC4: TC4, TerminalBlock_Phoenix:TerminalBlock_Phoenix_PT-1,5-2-3.5_1x02_P3.50mm_Horizontal, symbol Custom:Conn2pin
- removed J_TC5: TC5, TerminalBlock_Phoenix:TerminalBlock_Phoenix_PT-1,5-2-3.5_1x02_P3.50mm_Horizontal, symbol Custom:Conn2pin
- removed J_TC6: TC6, TerminalBlock_Phoenix:TerminalBlock_Phoenix_PT-1,5-2-3.5_1x02_P3.50mm_Horizontal, symbol Custom:Conn2pin
- removed J_TC7: TC7, TerminalBlock_Phoenix:TerminalBlock_Phoenix_PT-1,5-2-3.5_1x02_P3.50mm_Horizontal, symbol Custom:Conn2pin
- removed J_TC8: TC8, TerminalBlock_Phoenix:TerminalBlock_Phoenix_PT-1,5-2-3.5_1x02_P3.50mm_Horizontal, symbol Custom:Conn2pin
- removed Q_PMOS: AO3401A, Package_TO_SOT_SMD:SOT-23, symbol Custom:PMOS
- added C1, C10, C11, C12, C13, C14, C15, C16, C17, C18, C19, C20, C21, C22, C23, C24, C25, C26, C3, C4, C6, C7, C8, C9: 100nF, Capacitor_SMD:C_0805_2012Metric, symbol Custom:C_0805
- added C2, C5: 100uF/25V, Capacitor_THT:CP_Radial_D6.3mm_P2.50mm, symbol Custom:C_Elec
- added D1: SMBJ18A, Diode_SMD:D_SMB, symbol Custom:TVS
- added D2, D3, D4, D5: SS14, Diode_SMD:D_SMA, symbol Custom:SS14
- added D6: BZX84-C5V1, Diode_SMD:D_SOD-323, symbol Custom:Zener
- added D7, D8, D9: BZX84-C3V3, Diode_SMD:D_SOD-323, symbol Custom:Zener
- added J1: PWR_IN_12V, TerminalBlock_Phoenix:TerminalBlock_Phoenix_MKDS-1,5-2_1x02_P5.08mm_Horizontal, symbol Custom:PwrConn
- added J10: RPM_IN, TerminalBlock_Phoenix:TerminalBlock_Phoenix_PT-1,5-2-3.5_1x02_P3.50mm_Horizontal, symbol Custom:Conn2pin
- added J11: DIG1, TerminalBlock_Phoenix:TerminalBlock_Phoenix_PT-1,5-2-3.5_1x02_P3.50mm_Horizontal, symbol Custom:Conn2pin
- added J12: DIG2, TerminalBlock_Phoenix:TerminalBlock_Phoenix_PT-1,5-2-3.5_1x02_P3.50mm_Horizontal, symbol Custom:Conn2pin
- added J13: DIG3, TerminalBlock_Phoenix:TerminalBlock_Phoenix_PT-1,5-2-3.5_1x02_P3.50mm_Horizontal, symbol Custom:Conn2pin
- added J14: OUT1_FAN, TerminalBlock_Phoenix:TerminalBlock_Phoenix_PT-1,5-2-3.5_1x02_P3.50mm_Horizontal, symbol Custom:Conn2pin
- added J15: OUT2_PUMP, TerminalBlock_Phoenix:TerminalBlock_Phoenix_PT-1,5-2-3.5_1x02_P3.50mm_Horizontal, symbol Custom:Conn2pin
- added J16: OUT3_SHIFT_LIGHT, TerminalBlock_Phoenix:TerminalBlock_Phoenix_PT-1,5-2-3.5_1x02_P3.50mm_Horizontal, symbol Custom:Conn2pin
- added J17: OUT4_SPARE, TerminalBlock_Phoenix:TerminalBlock_Phoenix_PT-1,5-2-3.5_1x02_P3.50mm_Horizontal, symbol Custom:Conn2pin
- added J18: ANA1, TerminalBlock_Phoenix:TerminalBlock_Phoenix_PT-1,5-2-3.5_1x02_P3.50mm_Horizontal, symbol Custom:Conn2pin
- added J19: ANA2, TerminalBlock_Phoenix:TerminalBlock_Phoenix_PT-1,5-2-3.5_1x02_P3.50mm_Horizontal, symbol Custom:Conn2pin
- added J2: TC1, TerminalBlock_Phoenix:TerminalBlock_Phoenix_PT-1,5-2-3.5_1x02_P3.50mm_Horizontal, symbol Custom:Conn2pin
- added J20: NTC1, TerminalBlock_Phoenix:TerminalBlock_Phoenix_PT-1,5-2-3.5_1x02_P3.50mm_Horizontal, symbol Custom:Conn2pin
- added J21: NTC2, TerminalBlock_Phoenix:TerminalBlock_Phoenix_PT-1,5-2-3.5_1x02_P3.50mm_Horizontal, symbol Custom:Conn2pin
- added J22: NTC3, TerminalBlock_Phoenix:TerminalBlock_Phoenix_PT-1,5-2-3.5_1x02_P3.50mm_Horizontal, symbol Custom:Conn2pin
- added J23: NTC4, TerminalBlock_Phoenix:TerminalBlock_Phoenix_PT-1,5-2-3.5_1x02_P3.50mm_Horizontal, symbol Custom:Conn2pin
- added J24: GPS_MODULE, TerminalBlock_Phoenix:TerminalBlock_Phoenix_PT-1,5-4-3.5_1x04_P3.50mm_Horizontal, symbol Custom:Conn4pin
- added J25: NEOPIXEL_WS2812B, TerminalBlock_Phoenix:TerminalBlock_Phoenix_PT-1,5-3-3.5_1x03_P3.50mm_Horizontal, symbol Custom:Conn3pin
- added J26: EXPANSION, Connector_PinHeader_2.54mm:PinHeader_1x06_P2.54mm_Vertical, symbol Custom:Conn6pin
- added J3: TC2, TerminalBlock_Phoenix:TerminalBlock_Phoenix_PT-1,5-2-3.5_1x02_P3.50mm_Horizontal, symbol Custom:Conn2pin
- added J4: TC3, TerminalBlock_Phoenix:TerminalBlock_Phoenix_PT-1,5-2-3.5_1x02_P3.50mm_Horizontal, symbol Custom:Conn2pin
- added J5: TC4, TerminalBlock_Phoenix:TerminalBlock_Phoenix_PT-1,5-2-3.5_1x02_P3.50mm_Horizontal, symbol Custom:Conn2pin
- added J6: TC5, TerminalBlock_Phoenix:TerminalBlock_Phoenix_PT-1,5-2-3.5_1x02_P3.50mm_Horizontal, symbol Custom:Conn2pin
- added J7: TC6, TerminalBlock_Phoenix:TerminalBlock_Phoenix_PT-1,5-2-3.5_1x02_P3.50mm_Horizontal, symbol Custom:Conn2pin
- added J8: TC7, TerminalBlock_Phoenix:TerminalBlock_Phoenix_PT-1,5-2-3.5_1x02_P3.50mm_Horizontal, symbol Custom:Conn2pin
- added J9: TC8, TerminalBlock_Phoenix:TerminalBlock_Phoenix_PT-1,5-2-3.5_1x02_P3.50mm_Horizontal, symbol Custom:Conn2pin
- added L1: 10uH, Inductor_SMD:L_1210_3225Metric, symbol Custom:Inductor
- added LED1: GREEN_0805, LED_SMD:LED_0805_2012Metric, symbol Custom:LED_0805
- added Q5: AO3401A, Package_TO_SOT_SMD:SOT-23, symbol Custom:PMOS
- added R1: 1.5k, Resistor_SMD:R_0805_2012Metric, symbol Custom:R_0805
- added R10, R11, R14, R15, R16, R17, R22, R3, R4, R5, R6, R7, R8, R9: 10k, Resistor_SMD:R_0805_2012Metric, symbol Custom:R_0805
- added R12, R13: 15k, Resistor_SMD:R_0805_2012Metric, symbol Custom:R_0805
- added R18, R19, R20, R21: 100, Resistor_SMD:R_0805_2012Metric, symbol Custom:R_0805
- added R2: 270, Resistor_SMD:R_0805_2012Metric, symbol Custom:R_0805
- added R23: 100k, Resistor_SMD:R_0805_2012Metric, symbol Custom:R_0805
- added R24: 24.9k, Resistor_SMD:R_0805_2012Metric, symbol Custom:R_0805
- added R25: 300, Resistor_SMD:R_0805_2012Metric, symbol Custom:R_0805
- added R26: 1k, Resistor_SMD:R_0805_2012Metric, symbol Custom:R_0805
- added SW1: RESET, Button_Switch_THT:SW_PUSH_6mm_H5mm, symbol Custom:SW_Tactile
- added TP1: +12V, TestPoint:TestPoint_Pad_D1.5mm, symbol Custom:TestPad
- added TP10: RPM_IN, TestPoint:TestPoint_Pad_D1.5mm, symbol Custom:TestPad
- added TP2: +5V, TestPoint:TestPoint_Pad_D1.5mm, symbol Custom:TestPad
- added TP3: +3V3, TestPoint:TestPoint_Pad_D1.5mm, symbol Custom:TestPad
- added TP4: GND, TestPoint:TestPoint_Pad_D1.5mm, symbol Custom:TestPad
- added TP5: SPI_MOSI, TestPoint:TestPoint_Pad_D1.5mm, symbol Custom:TestPad
- added TP6: SPI_MISO, TestPoint:TestPoint_Pad_D1.5mm, symbol Custom:TestPad
- added TP7: SPI_SCK, TestPoint:TestPoint_Pad_D1.5mm, symbol Custom:TestPad
- added TP8: I2C_SDA, TestPoint:TestPoint_Pad_D1.5mm, symbol Custom:TestPad
- added TP9: I2C_SCL, TestPoint:TestPoint_Pad_D1.5mm, symbol Custom:TestPad
Connections:
- net +12V: now also J14.1 (Pin1), J15.1 (Pin1), J16.1 (Pin1), J17.1 (Pin1), Q5.1 (S)
- net +3V3: now also J24.4 (Pin4)
- net +5V: now also J25.3 (Pin3); no longer U12.5 (GND)
- net EXPN_P16: now also J26.6 (Pin6)
- net EXPN_P17: now also J26.5 (Pin5)
- net EXPN_P20: now also J26.4 (Pin4)
- net EXPN_P21: now also J26.3 (Pin3)
- net EXPN_P41: now also J26.2 (Pin2)
- net GND: now also J1.1 (+12V), J10.1 (Pin1), J11.1 (Pin1), J12.1 (Pin1), J13.1 (Pin1), J18.1 (Pin1), J19.1 (Pin1), J20.1 (Pin1), J21.1 (Pin1), J22.1 (Pin1), J23.1 (Pin1), J24.3 (Pin3), J25.1 (Pin1), J26.1 (Pin1)
- net GPS_RX: now also J24.2 (Pin2)
- net GPS_TX: now also J24.1 (Pin1)
- net LOAD1: now also J14.2 (Pin2)
- net LOAD2: now also J15.2 (Pin2)
- net LOAD3: now also J16.2 (Pin2)
- net LOAD4: now also J17.2 (Pin2)
- net NTC1: now also J20.2 (Pin2)
- net NTC2: now also J21.2 (Pin2)
- net NTC3: now also J22.2 (Pin2)
- net NTC4: now also J23.2 (Pin2)
- net TC1_M: now also J2.1 (Pin1)
- net TC1_P: now also J2.2 (Pin2)
- net TC2_M: now also J3.1 (Pin1)
- net TC2_P: now also J3.2 (Pin2)
- net TC3_M: now also J4.1 (Pin1)
- net TC3_P: now also J4.2 (Pin2)
- net TC4_M: now also J5.1 (Pin1)
- net TC4_P: now also J5.2 (Pin2)
- net TC5_M: now also J6.1 (Pin1)
- net TC5_P: now also J6.2 (Pin2)
- net TC6_M: now also J7.1 (Pin1)
- net TC6_P: now also J7.2 (Pin2)
- net TC7_M: now also J8.1 (Pin1)
- net TC7_P: now also J8.2 (Pin2)
- net TC8_M: now also J9.1 (Pin1)
- net TC8_P: now also J9.2 (Pin2)
- net VBAT_12V_IN: now also J1.2 (GND)
- net VBAT_FUSED: now also Q5.3 (D)
- net BOOT renamed BOOT_LMR
- net EXPN_P2 renamed STATUS_LED
- net NEO_5V renamed NEO_5V_BUF
- net RPM_SIG renamed RPM_LED
- new net ANA1_RAW: J18.2 (Pin2)
- new net ANA2_RAW: J19.2 (Pin2)
- new net DIG1_RAW: J11.2 (Pin2)
- new net DIG2_RAW: J12.2 (Pin2)
- new net DIG3_RAW: J13.2 (Pin2)
- new net NEO_DATA: J25.2 (Pin2)
- new net RPM_RAW: J10.2 (Pin2)
- new net SW_LMR: U12.5 (GND)
Other:
- note added: "+3V3, GND, GPS_TX->Teensy_RX(p34), Teensy_TX(p35)->GPS_RX"
- note added: "0-5V sensors -> R(10k)/R(15k) divider -> Teensy A0-A1 (p14-15)"
- note added: "10k top / 15k bottom = 5V -> 3.0V at ADC"
- note added: "5 unused Teensy pins on J26: p16, p17, p20, p21, p41 + GND"
- note added: "6N137 output -> R3(10k pull-up) -> Teensy p30"
- note added: "ANALOG IN (0-5V) + dividers"
- note added: "After F1 PTC fuse (~500mA)"
- note added: "After Q5 PMOS + D1 SMBJ18A TVS clamp"
- note added: "Buffers 2-4: OE tied to VCC (disabled)"
- note added: "Coil(-) -> R1(1.5k) -> D6(5.1V Zener) -> R2(270) -> 6N137"
- note added: "DIG1-3: R(10k) series + D(3.3V Zener) + C(100nF) + R(10k) pull-up"
- note added: "FB: 5V x 24.9k/(100k+24.9k) = 0.994V (Vref=1.0V)"
- note added: "GPS TX -> Teensy p34 Serial8 RX (4800/9600 baud NMEA)"
- note added: "K-type thermocouple T+/T- -> MAX31855 (EGT/CHT)"
- note added: "LMR33630Q1 — BUCK 12V to 5V 3A (automotive)"
- note added: "MAX31855 x 8 — THERMOCOUPLE ADC (SPI0)"
- note added: "MOSFET OUTPUTS x 4 (AO3400A N-ch + SS14 flyback)"
- note added: "MOSFET drain -> SS14 Schottky to +12V (flyback) + J_OUTx"
- note added: "NEO_3V3(p36) -> 1A -> 1Y(5V) -> R25(300) -> J25"
- note added: "NET LEGEND — v0.5.1 (complete with discretes)"
- note added: "NTC + R(10k) pull-up to 3V3 -> Teensy A8-A11 (p22-25)"
- note added: "R1(1.5k) -> D6(5.1V Zener) -> R2(270) -> 6N137 LED"
- note added: "R18-R21: 100ohm gate resistors | D2-D5: SS14 flyback"
- note added: "RESET BUTTON (6mm tactile)"
- note added: "RPM: Two-stage protection + 6N137 fast opto"
- note added: "RPM_RAW:"
- note added: "STATUS LED (p2, green 0805)"
- note added: "STATUS_LED:"
- note added: "SW1 tactile button -> Teensy RST pin -> GND"
- note added: "Switch -> R(10k) -> D(3.3V Zener) + C(100nF) + R(10k PU) -> p31-33"
- note added: "TEENSY 4.1 — MICROCONTROLLER (v0.5.1)"
- note added: "TEENSY_RST:"
- note added: "TEST PADS (TP1–TP10)"
- note added: "THERMOCOUPLE CONNECTORS J2–J9"
- note added: "TVS SMBJ18A: +12V to GND | PMOS gate: R22 10k to GND"
- note added: "Teensy internal reg ~250mA (LIS3DH, MAX31855, 6N137, logic)"
- note added: "Teensy p0 -> WIZ850io SCSn"
- note added: "Teensy p10,9,8,7,6,5,4,3 -> MAX31855 #0-7"
- note added: "Teensy p11/12/13 -> MAX31855x8 (SPI0, main bus)"
- note added: "Teensy p18 (Wire SDA) <-> LIS3DH SDA"
- note added: "Teensy p19 (Wire SCL) <-> LIS3DH SCL"
- note added: "Teensy p2 -> R26(1k) -> LED1(green 0805) -> GND"
- note added: "Teensy p26/1/27 <-> WIZ850io (SPI1, second bus)"
- note added: "Teensy p29 -> WIZ850io RSTn"
- note added: "Teensy p35 Serial8 TX -> GPS RX (bidirectional v0.5)"
- note added: "Teensy p36 -> 74AHCT125D buf1 -> R25(300) -> NeoPixel"
- note added: "Teensy p37-40 -> R(100) -> AO3400A gate (fan/pump/light/spare)"
- note added: "U12 LMR33630Q1 buck: L1(10uH), C1-C5, R23/R24 FB divider"
- note added: "VBAT_12V_IN -> PTC -> VBAT_FUSED -> PMOS(S->D) -> +12V"
- note added: "Vehicle 10-16V at J1 (5.08mm screw terminal)"
- note added: "WIZ850io INTn -> Teensy p28"
- note added: "p16, p17, p20, p21, p41 + GND"
- note removed: "+3V3, GND, GPS_TX→Teensy_RX(p34), Teensy_TX(p35)→GPS_RX"
- note removed: "0-5V sensors → Teensy A0-A1 (p14-15) via 10k/15k divider"
- note removed: "10k/15k divider to 3.3V"
- note removed: "6 unused Teensy pins on J_EXP header (p2,p16,p17,p20,p21,p41)"
- note removed: "ANALOG IN (0-5V)"
- note removed: "Add: L_out, C_in, C_out, R-divider for 5V"
- note removed: "After P-ch MOSFET reverse protect + SMBJ18A TVS clamp"
- note removed: "After PTC resettable fuse (~500mA)"
- note removed: "BOM v0.5:"
- note removed: "Buffers 2-4: OE tied to VCC (disabled, NC inputs/outputs)"
- note removed: "Coil/tacho → 270ohm → 6N137 LED → Teensy p30 (fast opto)"
- note removed: "DIG1-3: 10k series + 3.3V Zener + 100nF to GND + 10k pullup to 3V3"
- note removed: "GPS TX → Teensy p34 Serial8 RX (4800/9600 baud NMEA)"
- note removed: "J_RPM: 270ohm series + 5.1V Zener clamp before 6N137 LED"
- note removed: "K-type thermocouple T+/T- → MAX31855 (EGT/CHT/oil/coolant)"
- note removed: "LMR33630Q1 12V→5V 3A buck (Teensy VIN, GPS, NeoPixel)"
- note removed: "LMR33630Q1 — BUCK 12V→5V 3A (automotive)"
- note removed: "MAX31855 × 8 — THERMOCOUPLE ADC (SPI0)"
- note removed: "MOSFET OUTPUTS × 4 (AO3400A N-ch + SS14 flyback)"
- note removed: "MOSFET drain → SS14 Schottky to +12V (flyback) + J_OUTx"
- note removed: "NEO_3V3(p36) → 1A → 1Y(5V) → J_NEO data | OE1 tied to GND"
- note removed: "NET LEGEND — v0.5"
- note removed: "NTC 10k pull-up to 3V3 → Teensy A8-A11 (p22-25)"
- note removed: "OUT1=FAN OUT2=PUMP OUT3=SHIFT-LIGHT OUT4=SPARE"
- note removed: "RPM: 6N137 fast opto | DIG1-3: RC filter + Zener (see notes)"
- note removed: "Switch → 10k → Zener 3.3V + 100nF + 10k pullup → Teensy p31-33"
- note removed: "TEENSY 4.1 — MICROCONTROLLER (v0.5)"
- note removed: "THERMOCOUPLE CONNECTORS J_TC1–J_TC8"
- note removed: "TVS SMBJ18A: VBAT_PROT to GND | PMOS gate: GND via 10k"
- note removed: "Teensy internal reg ~250mA (LIS3DH, MAX31855, logic)"
- note removed: "Teensy p0 → WIZ850io SCSn"
- note removed: "Teensy p10,9,8,7,6,5,4,3 → MAX31855 #0-7"
- note removed: "Teensy p11/12/13 → MAX31855×8 (SPI0, main bus)"
- note removed: "Teensy p18 (Wire SDA) ↔ LIS3DH SDA"
- note removed: "Teensy p19 (Wire SCL) ↔ LIS3DH SCL"
- note removed: "Teensy p26/1/27 ↔ WIZ850io (SPI1, second bus)"
- note removed: "Teensy p29 → WIZ850io RSTn"
- note removed: "Teensy p35 Serial8 TX → GPS RX (bidirectional v0.5)"
- note removed: "Teensy p36 3.3V data → 74AHCT125D buf1 → 5V → NeoPixel"
- note removed: "Teensy p37-40 → 100ohm → AO3400A gate (fan/pump/light/spare)"
- note removed: "VBAT_12V_IN → PTC → VBAT_FUSED → PMOS(S→D) → VBAT_PROT(=+12V)"
- note removed: "Vehicle 10-16V input at J_PWR (5.08mm screw terminal)"
- note removed: "WIZ850io INTn → Teensy p28"
- note removed: "WIZ850io · LMR33630-Q1 · 6N137 · 74AHCT125D · PMOS · PTC · SS14"
- note removed: "p2, p16, p17, p20, p21, p41"
